Commit message: updating with visual indicators for mujoco

File: resources/robots/pointfoot/WF_TRON1A/urdf/robot.urdf (robot description, URDF)
Before this commit: robot wheel_biped, 10 links, 9 joints
Links:
- added link world
Joints:
- added joint base_free_joint: type floating, parent world, child base_Link, origin xyz=0 0 0 rpy=0 0 0
